File: PCB/VeraHDMI/jbVeraHDMI.sch (KiCad schematic (older format))
At the start: 70 parts, among them J2 Prog, J4 MercuryII-L, J5 MercuryII-R, J7 JTAG, U1 ICE40UP5K-SG48ITR50, U11 TFP410PAP, U12 SN74CB3T16210, U2 74AHC00PW, U3 LTC3406BES5-1.2, U4 74CBTLV3126PW,118, U6 WM8524CGEDT, U7 W25Q16JVSNIQ, U8 ATF1502AS-xAx44, X1 SG5032CAN_25.000000M-TJGA3

Commit message: Vera HDMI final updates, PCB's ordered.
Parts:
- C14: value 1u -> 1uF
- C29, C30: value .1uF -> 100nF
Changed lines of the file:
@@
 P 10750 5300
 F 0 "C14" V 10521 5300 50  0000 C CNN
-F 1 "1u" V 10612 5300 50  0000 C CNN
+F 1 "1uF" V 10612 5300 50  0000 C CNN
 F 2 "Capacitor_SMD:C_0603_1608Metric_Pad1.08x0.95mm_HandSolder" H 10750 5300 50  0001 C CNN
 F 3 "~" H 10750 5300 50  0001 C CNN
@@
 P 14300 3700
 F 0 "C29" V 14250 3550 50  0000 L CNN
-F 1 ".1uF" V 14250 3750 50  0000 L CNN
+F 1 "100nF" V 14250 3750 50  0000 L CNN
 F 2 "Capacitor_SMD:C_0603_1608Metric_Pad1.08x0.95mm_HandSolder" H 14300 3700 50  0001 C CNN
 F 3 "~" H 14300 3700 50  0001 C CNN
@@
 P 14450 3700
 F 0 "C30" V 14400 3550 50  0000 L CNN
-F 1 ".1uF" V 14400 3750 50  0000 L CNN
+F 1 "100nF" V 14400 3750 50  0000 L CNN
 F 2 "Capacitor_SMD:C_0603_1608Metric_Pad1.08x0.95mm_HandSolder" H 14450 3700 50  0001 C CNN
 F 3 "~" H 14450 3700 50  0001 C CNN
