File: PCB/VeraHDMI/jbVeraHDMI.kicad_pcb (KiCad board)
At the start: 4 copper layers, 26.6 x 84.3 mm, 70 parts, among them J2 Prog, J4 MercuryII-L, J5 MercuryII-R, J7 JTAG, U1 ICE40UP5K-SG48ITR50, U11 TFP410PAP, U12 SN74CB3T16210, U2 74AHC00PW, U3 LTC3406BES5-1.2, U4 74CBTLV3126PW,118, U6 WM8524CGEDT, U7 W25Q16JVSNIQ, U8 ATF1502AS-xAx44, X1 SG5032CAN_25.000000M-TJGA3

Commit message: Updates
Other:
- net class Default removed
