File: PCB/JBX16/JBX16.sch (KiCad schematic (older format))
At the start: 157 parts, among them J1 ROMWR, J10 MercuryII_B, J11 AudioOut, J12 ATX-20, J13 HDMI_A_1.4, J14 UART-A, J15 UART-B, J16 Micro_SD_Card, J17 User Port, J18 SNES P3/P4, J2 DIN-6, J3 JTAG, J4 SNES P1, J5 TinyISP, J6 IRQ/NMI, J7 Keyboard/Mouse, J8 SNES P2, J9 MercuryII_A, SW1 POWER, SW2 RESET, SW3 NMI, U1 WD65C02, U10 74HC245, U11 74HC245, U12 74HC245, U13 74HC245, U14 SC28L92A1A, U15 ATtiny861-20PU, U16 WD65C22, U17 WD65C22, U18 YM2151, U19 YM3012, U2 SN7406, U20 TL074, U21 TL072, U3 SST39SF040, U4 AS6C1008-55PCN, U5 AS6C4008-55PCN, U6 AS6C4008-55PCN, U7 AS6C4008-55PCN, U8 AS6C4008-55PCN, U9 ATF1508, X1 16mhz, X2 8mhz, X3 3.579545MHz

Commit message: Updates to layout
Parts:
- removed J12: ATX-20, Connector_Molex:Molex_Mini-Fit_Jr_5566-20A_2x10_P4.20mm_Vertical, symbol Connector:ATX-20
- added H10: H, MountingHole:MountingHole_3.2mm_M3_ISO7380_Pad, symbol Mechanical:MountingHole
- added J12, J20, J21: Conn_02x36_Odd_Even, Connector_PinSocket_2.54mm:PinSocket_2x36_P2.54mm_Vertical, symbol Connector_Generic:Conn_02x36_Odd_Even
- added J19: ATX-24, Connector_Molex:Molex_Mini-Fit_Jr_5566-24A_2x12_P4.20mm_Vertical, symbol Connector:ATX-24
- added J28: Conn_02x30_Odd_Even, Connector_PinSocket_2.54mm:PinSocket_2x30_P2.54mm_Vertical, symbol Connector_Generic:Conn_02x30_Odd_Even
- added R25: 1K, Resistor_THT:R_Axial_DIN0204_L3.6mm_D1.6mm_P5.08mm_Horizontal, symbol Device:R_Small
- added R26, R27: DNI, Resistor_THT:R_Axial_DIN0204_L3.6mm_D1.6mm_P5.08mm_Horizontal, symbol Device:R_US
Connections:
- net labels added: +12, +3.3, +5, -12, RD#, WR#, bc, mp
- net labels removed: CLKWR, OELOW, UADATDIR
- wire segments 411 -> 446
Other:
- note added: "EXPANSION"
- note added: "vc"
- moved on the sheet: C45, C46, C47, C48, C49, C50, C51, C52, C53, C54, C55, H1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

Commit message: Many Updates
Parts:
- removed H10: H, MountingHole:MountingHole_3.2mm_M3_ISO7380_Pad, symbol Mechanical:MountingHole
- removed J10: MercuryII_B, Connector_PinSocket_2.54mm:PinSocket_1x32_P2.54mm_Vertical, symbol Connectors:Conn_01x32_Female
- removed J14: UART-A, Connector_PinSocket_2.54mm:PinSocket_1x06_P2.54mm_Vertical, symbol Connector:Conn_01x06_Male
- removed J9: MercuryII_A, Connector_PinSocket_2.54mm:PinSocket_1x32_P2.54mm_Vertical, symbol Connectors:Conn_01x32_Female
- added BT1: CR2032, Battery:BatteryHolder_Keystone_1060_1x2032, symbol Device:Battery_Cell
- added C65, C66, C67, C68, C69, C70, C71, C72, C73, C74, C75, C77, C78, C79, C80, C81, C82: 330pF, Capacitor_THT:C_Disc_D3.0mm_W1.6mm_P2.50mm, symbol Device:C_Small
- added C76: .1uF, Capacitor_THT:C_Disc_D3.0mm_W1.6mm_P2.50mm, symbol Device:C_Small
- added C83, C84: 9pF, Capacitor_THT:C_Disc_D3.0mm_W1.6mm_P2.50mm, symbol Device:C_Small
- added D10, D11, D12, D13, D14, D15, D2, D20, D3, D4, D9: BLUE, LED_SMD:LED_0805_2012Metric_Pad1.15x1.40mm_HandSolder, symbol Device:LED_Small
- added D16: AMBER, LED_SMD:LED_0805_2012Metric_Pad1.15x1.40mm_HandSolder, symbol Device:LED_Small
- added D19, D23, D24, D25, D26: GREEN, LED_SMD:LED_0805_2012Metric_Pad1.15x1.40mm_HandSolder, symbol Device:LED_Small
- added D27: 1N4148, Diode_THT:D_T-1_P5.08mm_Horizontal, symbol Diode:1N4148
- added J22: Conn_02x05_Odd_Even, Connector_PinSocket_2.54mm:PinSocket_2x05_P2.54mm_Vertical, symbol Connector_Generic:Conn_02x05_Odd_Even
- added J9: UART-A, Connector_PinSocket_2.54mm:PinSocket_1x06_P2.54mm_Vertical, symbol Connector:Conn_01x06_Male
- added Q1, Q2, Q3, Q4: BC327, Package_TO_SOT_THT:TO-92_Inline, symbol Transistor_BJT:BC307
- added R28, R29, R30, R31, R32, R33, R34, R35, R36, R37, R38, R41, R42, R45, R46, R47, R48, R49, R50, R51, R52: 1K, Resistor_SMD:R_0805_2012Metric_Pad1.20x1.40mm_HandSolder, symbol Device:R_Small
- added R43, R44, R55, R56, R57, R58: 47K, Resistor_SMD:R_0805_2012Metric_Pad1.20x1.40mm_HandSolder, symbol Device:R_Small
- added R53, R54: 1K, Resistor_THT:R_Axial_DIN0204_L3.6mm_D1.6mm_P5.08mm_Horizontal, symbol Device:R_Small
- added U22: MCP7940N-xP, Package_DIP:DIP-8_W7.62mm, symbol Timer:MCP7940N-xP
- added U23: MercuryII-FPGA, JBCustoms:MercuryII_FPGA, symbol JBX16Customs:MercuryII-FPGA
- added Y1: 32.768KHz, Crystal:Crystal_C26-LF_D2.1mm_L6.5mm_Horizontal, symbol Device:Crystal_Small
Connections:
- net labels added: SD_MISO, SD_MOSI, SD_SCK, SD_SSEL
- net labels removed: UAEN, s1CTS, s1RTS, s1RX, s1TX, sd_CLK, sd_CMD, sd_D0, sd_D1, sd_D2, sd_D3
- wire segments 446 -> 577
- no-connect marks 1 -> 46
Other:
- note added: "3.6mA current to CPLD when low. \n"
- note added: "EXPANSION BUS"
- note added: "Headers / Misc."
- note added: "Real Time Clock"
- note added: "SYSTEM STATUS LEDS"
- note removed: "EXPANSION"
- moved on the sheet: C22, C23, C28, C29, C30, C31, C32, C36, C37, C38, C39, C40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

Commit message: Board build progress.
Parts:
- removed RN1: 4.7K, Resistor_THT:R_Array_SIP8, symbol Device:R_Network07_US
- added JP3: VSEL, Jumper:SolderJumper-3_P1.3mm_Open_Pad1.0x1.5mm_NumberLabels, symbol Jumper:SolderJumper_3_Open
- added Q5, Q6: BC327, Package_TO_SOT_THT:TO-92_Inline, symbol Transistor_BJT:BC307
- added R39: 10R, Resistor_THT:R_Axial_DIN0204_L3.6mm_D1.6mm_P5.08mm_Horizontal, symbol Device:R_Small
- added R40: 1K, Resistor_THT:R_Axial_DIN0204_L3.6mm_D1.6mm_P5.08mm_Horizontal, symbol Device:R_Small
- added RN1: 4.7K, Resistor_THT:R_Array_SIP6, symbol Device:R_Network05_US
Connections:
- net labels removed: ABORT, MLB, SOB, SYNC, V0CA1, V0CA2, VPS2KCLK, VPS2KDAT, VPS2MCLK, VPS2MDAT
- wire segments 577 -> 586
- no-connect marks 46 -> 56
Other:
- note added: "Misc."
- note added: "SYSTEM STATUS"
- note added: "Spike/EMI Protection"
- note removed: "Headers / Misc."
- note removed: "SYSTEM STATUS LEDS"
- note removed: "Spike Protection"
- moved on the sheet: C2, C22, C23, C24, C25, C26, C27, C28, C33, C34, C35, C56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

Commit message: Final Changes, PCB's ordered
Parts:
- removed C28, C39: .1uF, Capacitor_THT:C_Disc_D3.0mm_W1.6mm_P2.50mm, symbol Device:C
- removed C38: 1uF, Capacitor_THT:C_Disc_D3.0mm_W1.6mm_P2.50mm, symbol Device:C
- removed H7, H8, H9: H, MountingHole:MountingHole_3.2mm_M3_ISO7380_Pad, symbol Mechanical:MountingHole
- removed J15: UART-B, Connector_PinSocket_2.54mm:PinSocket_1x06_P2.54mm_Vertical, symbol Connector:Conn_01x06_Male
- removed J9: UART-A, Connector_PinSocket_2.54mm:PinSocket_1x06_P2.54mm_Vertical, symbol Connector:Conn_01x06_Male
- removed U14: SC28L92A1A, Package_LCC:PLCC-44_THT-Socket, symbol JBX16Customs:SC28L92A1A
- removed X2: 8mhz, Oscillator:Oscillator_DIP-8, symbol Oscillator:CXO_DIP8
- added C28, C38: 10uF, Capacitor_THT:CP_Radial_D5.0mm_P2.00mm, symbol Device:CP1_Small
- added C85, C86: 2700pF, Capacitor_THT:C_Disc_D3.0mm_W1.6mm_P2.50mm, symbol Device:C
- added C87, C88, C91, C92: 1uF, Capacitor_THT:C_Disc_D3.0mm_W1.6mm_P2.50mm, symbol Device:C
- added C89, C90: 3300pF, Capacitor_THT:C_Disc_D3.0mm_W1.6mm_P2.50mm, symbol Device:C
- added J10: MercAudioEn, Connector_PinHeader_2.54mm:PinHeader_2x03_P2.54mm_Vertical, symbol Connector_Generic:Conn_02x03_Odd_Even
- added J14: VeraAudioEn, Connector_PinHeader_2.54mm:PinHeader_2x03_P2.54mm_Vertical, symbol Connector_Generic:Conn_02x03_Odd_Even
- added J15: frontPannel, Connector_PinHeader_2.54mm:PinHeader_2x05_P2.54mm_Vertical, symbol Connector_Generic:Conn_02x05_Odd_Even
- added J23: Conn_02x04_Odd_Even, Connector_PinHeader_2.54mm:PinHeader_2x04_P2.54mm_Vertical, symbol Connector_Generic:Conn_02x04_Odd_Even
- added J9: AuxIn, Connector_PinHeader_2.54mm:PinHeader_1x03_P2.54mm_Vertical, symbol Connector:Conn_01x03_Male
- added Q7: BC327, Package_TO_SOT_THT:TO-92_Inline, symbol Transistor_BJT:BC307
- added R59, R60, R61, R62, R63, R64, R65, R66, R69, R70, R71, R72: 10K, Resistor_THT:R_Axial_DIN0204_L3.6mm_D1.6mm_P5.08mm_Horizontal, symbol Device:R_Small
- added R67, R68: 23K, Resistor_THT:R_Axial_DIN0204_L3.6mm_D1.6mm_P5.08mm_Horizontal, symbol Device:R_Small
- added R73, R74, R75: 1K, Resistor_SMD:R_0805_2012Metric_Pad1.20x1.40mm_HandSolder, symbol Device:R_Small
- added U14: TL074, Package_DIP:DIP-14_W7.62mm_Socket, symbol Amplifier_Operational:TL074
- C36: value 1uF -> .1uF
- J1: footprint Connector_PinSocket_2.54mm:PinSocket_1x02_P2.54mm_Vertical -> Connector_PinHeader_2.54mm:PinHeader_1x02_P2.54mm_Vertical
- J22: footprint Connector_PinSocket_2.54mm:PinSocket_2x05_P2.54mm_Vertical -> Connector_PinHeader_2.54mm:PinHeader_2x05_P2.54mm_Vertical
Connections:
- net +12V: now also C22.1, C28.1, U14.4 (V+)
- net +5V: now also J17.26 (Pin_26), J23.1 (Pin_1), Q7.3 (E), R74.2; no longer C22.1, R36.1
- net -12V: now also C36.1, C38.2, U14.11 (V-)
- net 5VSB: now also D1.1 (K); no longer J19.9 (+5VSB)
- net CH1: now also R12.2; no longer U20.10 (+)
- net CH2: now also R20.2; no longer U20.12 (+)
- net GND: now also C36.2, D14.1 (K), U20.10 (+), U20.12 (+), C28.2, C38.1, C85.2, C86.2, C89.2, C90.2, J10.5 (Pin_5), J10.6 (Pin_6), J14.5 (Pin_5), J14.6 (Pin_6), J15.10 (Pin_10), J15.2 (Pin_2), J15.4 (Pin_4), J15.6 (Pin_6), J15.8 (Pin_8), J23.2 (Pin_2), J9.2 (Pin_2), U14.10 (+), U14.12 (+), U14.3 (+), U14.5 (+)
- net IRQ: now also U18.2 (IRQ); no longer D1.2 (A)
- net NMIBTN: now also J15.9 (Pin_9)
- net PWRBTN: now also J15.5 (Pin_5)
- net RSTBTN: now also J15.7 (Pin_7)
- net SRLEN: no longer D14.1 (K)
- net vDACL: now also J10.1 (Pin_1), J14.1 (Pin_1); no longer C36.2
- net vDACR: now also J10.2 (Pin_2), J14.2 (Pin_2)
- net at U9.80 (IO): now also R36.2
- net at C32.2, U20.8: now also R61.1; no longer U20.9 (-)
- net at C37.2, U20.14: now also R62.1; no longer U20.13 (-)
- net at C32.1: now also R65.2; no longer R12.2
- net at C37.1: now also R66.2; no longer R20.2
- net VERA_R: now reaches R21.2
- net VERA_R: now also C86.1, J14.4 (Pin_4)
- net at R18.2: now also J9.3 (Pin_3); no longer C36.1
- net MIXER_R: now reaches C41.2, R23.2, U21.2 (-)
- net MIXER_R: now also R18.1, R64.1, R66.1, R72.1; no longer R19.1, R20.1, R21.1
- net MIXER_L: now reaches C40.2, R22.2, R8.1, U21.6 (-)
- net MIXER_L: now also R63.1, R65.1, R71.1; no longer R12.1, R18.1
- net at D14.2 (A): now also R73.2; no longer R36.2
- net V0PB0: now reaches U16.10 (PB0)
- net V0PB0: now also J23.7 (Pin_7)
- net V0PB1: now reaches U16.11 (PB1)
- net V0PB1: now also J23.8 (Pin_8)
- net V0PB2: now reaches U16.12 (PB2)
- net V0PB2: now also J23.6 (Pin_6)
- net V0CB2: now reaches U16.19 (CB2)
- net V0CB2: now also J23.5 (Pin_5)
- net V0CA2: now reaches U16.39 (CA2)
- net V0CA2: now also J23.3 (Pin_3)
- net V0CA1: now reaches U16.40 (CA1)
- net V0CA1: now also J23.4 (Pin_4)
- net SH1: no longer names the net of U18.20 (SH1), U19.6 (SAM1)
- net SH2: no longer names the net of U18.19 (SH2), U19.5 (SAM2)
- net SO: no longer names the net of U18.21 (SO), U19.4 (SD)
- net YPHI1: no longer names the net of U18.23 (PHI1), U19.2 (PHI1)
- net sAUXL: no longer names the net of R8.2
- net sAUXL: now also J9.1 (Pin_1)
- net sAUXR renamed VERA_L
- net VERA_L: now also C85.1, J14.3 (Pin_3)
- new net: C87.2, R59.1, U14.1
- new net: R19.1, R59.2, U14.2 (-)
- new net: R21.1, R60.2, U14.6 (-)
- new net: C88.2, R60.1, U14.7
- new net: C91.2, R69.1, U14.8
- new net: R67.1, R69.2, U14.9 (-)
- new net: R68.1, R70.2, U14.13 (-)
- new net: C92.2, R70.1, U14.14
- new net: D1.2 (A), J19.9 (+5VSB)
- new net: C87.1, R63.2
- new net: R12.1, R61.2, U20.9 (-)
- new net: R20.1, R62.2, U20.13 (-)
- new net: C88.1, R64.2
- new net: C91.1, R71.2
- new net: C92.1, R72.2
- new net: J15.1 (Pin_1), R74.1
- new net: J15.3 (Pin_3), R75.1
- new net: Q7.2 (B), R36.1
- new net CPLDACT: Q7.1 (C), R73.1, R75.2
- new net MERC_L: C89.1, J10.3 (Pin_3), R67.2
- new net MERC_R: C90.1, J10.4 (Pin_4), R68.2
- no-connect marks 56 -> 39
Other:
- note removed: "UART"
- moved on the sheet: C29, C30, C31, C32, C37, C40, C41, C42, C43, C44, C45, C46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

Commit message: Notated bad circuits
5v rail leaking into RST bus through Q1, needs revision.
ATX Loading during power down is trash, do not use R39,R40,Q5,Q6
Parts:
- R46: value 1K -> 4.7K
Other:
- note added: "DNI, \nP-FET Fix?"
- note added: "failed ATX loading circuit. \nDo not install"
Changed lines of the file:
@@
 AR Path="/630B3D2B" Ref="R46"  Part="1"
 F 0 "R46" V 19000 10000 50  0000 L CNN
-F 1 "1K" V 19100 10000 50  0000 L CNN
+F 1 "4.7K" V 19050 9800 50  0000 L CNN
 F 2 "Resistor_SMD:R_0805_2012Metric_Pad1.20x1.40mm_HandSolder" H 19100 10050 50  0001 C CNN
 F 3 "~" H 19100 10050 50  0001 C CNN
@@
 Wire Wire Line
 	15650 3900 15700 3900
+Wire Notes Line style dash_dot rgb(255, 0, 0)
+	6650 10500 6650 9150
+Wire Notes Line style dash_dot rgb(255, 0, 0)
+	6650 9150 5150 9150
+Wire Notes Line style dash_dot rgb(255, 0, 0)
+	5150 9150 5150 10500
+Wire Notes Line style dash_dot rgb(255, 0, 0)
+	5150 10500 6650 10500
+Text Notes 5200 9400 0    50   ~ 0
+failed ATX loading circuit. \nDo not install
+Wire Notes Line style dash_dot rgb(255, 0, 0)
+	18600 10750 19250 10750
+Wire Notes Line style dash_dot rgb(255, 0, 0)
+	19250 10750 19250 9350
+Wire Notes Line style dash_dot rgb(255, 0, 0)
+	19250 9350 18600 9350
+Wire Notes Line style dash_dot rgb(255, 0, 0)
+	18600 9350 18600 10750
+Text Notes 18650 9500 0    50   ~ 0
+DNI, \nP-FET Fix?
 $EndSCHEMATC

Commit message: ATX Loading + RST FET + Activity FET
Removed ATX load circuit. Updated RST + Activity LED drivers from BJT to P-FET.
Parts:
- removed Q1, Q5, Q6, Q7: BC327, Package_TO_SOT_THT:TO-92_Inline, symbol Transistor_BJT:BC307
- removed R39: 10R, Resistor_THT:R_Axial_DIN0204_L3.6mm_D1.6mm_P5.08mm_Horizontal, symbol Device:R_Small
- removed R40: 1K, Resistor_THT:R_Axial_DIN0204_L3.6mm_D1.6mm_P5.08mm_Horizontal, symbol Device:R_Small
- added Q1, Q7: BS250, Package_TO_SOT_THT:TO-92_Inline, symbol Transistor_FET:BS250
- D23: value GREEN -> RED
- R46: value 4.7K -> 1K
Connections:
- net +5V: now also Q1.3 (S), Q7.3 (S)
- net CPLDACT: now also Q7.1 (D)
- net at R45.2: now also Q1.1 (D)
- net at R46.2: now also Q1.2 (G)
- net at R36.1: now also Q7.2 (G)
Other:
- note removed: "3.6mA current to CPLD when low. \n"
- note removed: "DNI, \nP-FET Fix?"
- note removed: "failed ATX loading circuit. \nDo not install"
- moved on the sheet: D23, R45, R46

Commit message: Updates
Parts:
- C25, C26, C27: symbol Device:CP1 -> JBX16-rescue:CP1-Device
- C28, C38, C44, C46, C49, C50, C53, C55: symbol Device:CP1_Small -> JBX16-rescue:CP1_Small-Device
- F1, F2, F3, F4: symbol Device:Polyfuse -> JBX16-rescue:Polyfuse-Device
- JP1: symbol Jumper:Jumper_3_Open -> JBX16-rescue:Jumper_3_Open-Jumper
- JP2: symbol Device:Jumper -> JBX16-rescue:Jumper-Device
- JP3: symbol Jumper:SolderJumper_3_Open -> JBX16-rescue:SolderJumper_3_Open-Jumper
- U15: symbol MCU_Microchip_ATtiny:ATtiny861-20PU -> JBX16-rescue:ATtiny861-20PU-MCU_Microchip_ATtiny
- U22: symbol Timer:MCP7940N-xP -> JBX16-rescue:MCP7940N-xP-Timer
