File: PCB/JBX16/JBX16.kicad_sch (KiCad schematic)
At the start: 263 parts

Commit message: PLCC Update for VP Fix
Parts:
- BT1: value (none) -> CR2032; footprint (none) -> Battery:BatteryHolder_Keystone_1060_1x2032
- C1, C10, C11, C12, C13, C14, C15, C16, C17, C18, C19, C2, C20, C21, C22, C24, C29, C3, C33, C34, C35, C36, C4, C45, C47, C48, C5, C51, C52, C54, C6, C7, C76, C8, C9: value (none) -> .1uF; footprint (none) -> Capacitor_THT:C_Disc_D3.0mm_W1.6mm_P2.50mm
- C23, C56, C57, C58, C59, C60, C61, C62, C63, C64, C65, C66, C67, C68, C69, C70, C71, C72, C73, C74, C75, C77, C78, C79, C80, C81, C82: value (none) -> 330pF; footprint (none) -> Capacitor_THT:C_Disc_D3.0mm_W1.6mm_P2.50mm
- C25, C26, C27: value (none) -> CP1; footprint (none) -> Capacitor_THT:CP_Radial_D10.0mm_P5.00mm
- C28, C38, C44, C46, C49, C50, C53, C55: value (none) -> 10uF; footprint (none) -> Capacitor_THT:CP_Radial_D5.0mm_P2.00mm
- C30, C31, C89, C90: value (none) -> 3300pF; footprint (none) -> Capacitor_THT:C_Disc_D3.0mm_W1.6mm_P2.50mm
- C32, C37, C42, C43, C87, C88, C91, C92: value (none) -> 1uF; footprint (none) -> Capacitor_THT:C_Disc_D3.0mm_W1.6mm_P2.50mm
- C40, C41: value (none) -> 1000pF; footprint (none) -> Capacitor_THT:C_Disc_D3.0mm_W1.6mm_P2.50mm
- C83, C84: value (none) -> 9pF; footprint (none) -> Capacitor_THT:C_Disc_D3.0mm_W1.6mm_P2.50mm
- C85, C86: value (none) -> 2700pF; footprint (none) -> Capacitor_THT:C_Disc_D3.0mm_W1.6mm_P2.50mm
- D1, D27, D5, D6, D7, D8: value (none) -> 1N4148; footprint (none) -> Diode_THT:D_T-1_P5.08mm_Horizontal
- D10, D11, D12, D13, D14, D15, D2, D20, D3, D4, D9: value (none) -> BLUE; footprint (none) -> LED_SMD:LED_0805_2012Metric_Pad1.15x1.40mm_HandSolder
- D16: value (none) -> AMBER; footprint (none) -> LED_SMD:LED_0805_2012Metric_Pad1.15x1.40mm_HandSolder
- D19, D24, D25, D26: value (none) -> GREEN; footprint (none) -> LED_SMD:LED_0805_2012Metric_Pad1.15x1.40mm_HandSolder
- D23: value (none) -> RED; footprint (none) -> LED_SMD:LED_0805_2012Metric_Pad1.15x1.40mm_HandSolder
- F1, F2, F3, F4: value (none) -> RUSBF185-AP; footprint (none) -> Fuse:Fuse_Littelfuse_395Series
- H1, H2, H3, H4, H5, H6: value (none) -> H; footprint (none) -> MountingHole:MountingHole_3.2mm_M3_ISO7380_Pad
- J1: value (none) -> ROMWR; footprint (none) -> Connector_PinHeader_2.54mm:PinHeader_1x02_P2.54mm_Vertical
- J10: value (none) -> MercAudioEn; footprint (none) -> Connector_PinHeader_2.54mm:PinHeader_2x03_P2.54mm_Vertical
- J11: value (none) -> AudioOut; footprint (none) -> Connector_Audio:Jack_3.5mm_CUI_SJ1-3533NG_Horizontal_CircularHoles
- J12, J20, J21: value (none) -> Conn_02x36_Odd_Even; footprint (none) -> Connector_PinSocket_2.54mm:PinSocket_2x36_P2.54mm_Vertical
- J13: value (none) -> HDMI_A_1.4; footprint (none) -> Connector_HDMI:HDMI_A_Kycon_KDMIX-SL1-NS-WS-B15_VerticalRightAngle
- J14: value (none) -> VeraAudioEn; footprint (none) -> Connector_PinHeader_2.54mm:PinHeader_2x03_P2.54mm_Vertical
- J15: value (none) -> frontPannel; footprint (none) -> Connector_PinHeader_2.54mm:PinHeader_2x05_P2.54mm_Vertical
- J16: value (none) -> Micro_SD_Card; footprint (none) -> Connector_Card:microSD_HC_Hirose_DM3AT-SF-PEJM5
- J17: value (none) -> User Port; footprint (none) -> Connector_PinHeader_2.54mm:PinHeader_2x13_P2.54mm_Vertical
- J18: value (none) -> SNES P3/P4; footprint (none) -> Connector_PinHeader_2.54mm:PinHeader_2x03_P2.54mm_Vertical
- J19: value (none) -> ATX-24; footprint (none) -> Connector_Molex:Molex_Mini-Fit_Jr_5566-24A_2x12_P4.20mm_Vertical
- J2: value (none) -> DIN-6; footprint (none) -> JBCustoms:DIN-6-IEC
- J22: value (none) -> Conn_02x05_Odd_Even; footprint (none) -> Connector_PinHeader_2.54mm:PinHeader_2x05_P2.54mm_Vertical
- J23: value (none) -> Conn_02x04_Odd_Even; footprint (none) -> Connector_PinHeader_2.54mm:PinHeader_2x04_P2.54mm_Vertical
- J28: value (none) -> Conn_02x30_Odd_Even; footprint (none) -> Connector_PinSocket_2.54mm:PinSocket_2x30_P2.54mm_Vertical
- J3: value (none) -> JTAG; footprint (none) -> Connector_PinHeader_2.54mm:PinHeader_2x05_P2.54mm_Vertical
- J4: value (none) -> SNES P1; footprint (none) -> JBCustoms:SNES
- J5: value (none) -> TinyISP; footprint (none) -> Connector_PinHeader_2.54mm:PinHeader_2x03_P2.54mm_Vertical
- J6: value (none) -> IRQ/NMI; footprint (none) -> Connector_PinHeader_2.54mm:PinHeader_1x03_P2.54mm_Vertical
- J7: value (none) -> Keyboard/Mouse; footprint (none) -> CX16:MD-60SM
- J8: value (none) -> SNES P2; footprint (none) -> JBCustoms:SNES
- J9: value (none) -> AuxIn; footprint (none) -> Connector_PinHeader_2.54mm:PinHeader_1x03_P2.54mm_Vertical
- JP1: value (none) -> ADC_VREF; footprint (none) -> Connector_PinHeader_2.54mm:PinHeader_1x03_P2.54mm_Vertical
- JP2: value (none) -> PSU_3.3V; footprint (none) -> Connector_PinHeader_2.54mm:PinHeader_1x02_P2.54mm_Vertical
- JP3: value (none) -> VSEL; footprint (none) -> Jumper:SolderJumper-3_P1.3mm_Open_Pad1.0x1.5mm_NumberLabels
- L1: value (none) -> 820uh; footprint (none) -> Inductor_THT:L_Axial_L7.0mm_D3.3mm_P12.70mm_Horizontal_Fastron_MICC
- Q1, Q7: value (none) -> BS250; footprint (none) -> Package_TO_SOT_THT:TO-92_Inline
- Q2, Q3, Q4: value (none) -> BC327; footprint (none) -> Package_TO_SOT_THT:TO-92_Inline
- R1, R10, R2, R25, R3, R4, R53, R54, R7, R9: value (none) -> 1K; footprint (none) -> Resistor_THT:R_Axial_DIN0204_L3.6mm_D1.6mm_P5.08mm_Horizontal
- R11, R15, R16, R18, R19, R21, R22, R23, R5, R59, R6, R60, R61, R62, R63, R64, R65, R66, R69, R70, R71, R72, R8: value (none) -> 10K; footprint (none) -> Resistor_THT:R_Axial_DIN0204_L3.6mm_D1.6mm_P5.08mm_Horizontal
- R12, R20: value (none) -> 40K; footprint (none) -> Resistor_THT:R_Axial_DIN0204_L3.6mm_D1.6mm_P5.08mm_Horizontal
- R13, R14, R17: value (none) -> 4.7K; footprint (none) -> Resistor_THT:R_Axial_DIN0204_L3.6mm_D1.6mm_P5.08mm_Horizontal
- R24: value (none) -> 100; footprint (none) -> Resistor_THT:R_Axial_DIN0204_L3.6mm_D1.6mm_P5.08mm_Horizontal
- R26, R27: value (none) -> DNI; footprint (none) -> Resistor_THT:R_Axial_DIN0204_L3.6mm_D1.6mm_P5.08mm_Horizontal
- R28, R29, R30, R31, R32, R33, R34, R35, R36, R37, R38, R41, R42, R45, R46, R47, R48, R49, R50, R51, R52, R73, R74, R75: value (none) -> 1K; footprint (none) -> Resistor_SMD:R_0805_2012Metric_Pad1.20x1.40mm_HandSolder
- R43, R44, R55, R56, R57, R58: value (none) -> 47K; footprint (none) -> Resistor_SMD:R_0805_2012Metric_Pad1.20x1.40mm_HandSolder
- R67, R68: value (none) -> 23K; footprint (none) -> Resistor_THT:R_Axial_DIN0204_L3.6mm_D1.6mm_P5.08mm_Horizontal
- RN1, RN3: value (none) -> 4.7K; footprint (none) -> Resistor_THT:R_Array_SIP6
- RN2: value (none) -> 4.7K; footprint (none) -> Resistor_THT:R_Array_SIP5
- SW1: value (none) -> POWER; footprint (none) -> Button_Switch_THT:SW_PUSH_6mm
- SW2: value (none) -> RESET; footprint (none) -> Button_Switch_THT:SW_PUSH_6mm
- SW3: value (none) -> NMI; footprint (none) -> Button_Switch_THT:SW_PUSH_6mm
- U1: value (none) -> WD65C02; footprint (none) -> Package_DIP:DIP-40_W15.24mm_Socket
- U10, U11, U12, U13: value (none) -> 74HC245; footprint (none) -> Package_DIP:DIP-20_W7.62mm_Socket
- U14, U20: value (none) -> TL074; footprint (none) -> Package_DIP:DIP-14_W7.62mm_Socket
- U15: value (none) -> ATtiny861-20PU; footprint (none) -> Package_DIP:DIP-20_W7.62mm_Socket
- U16, U17: value (none) -> WD65C22; footprint (none) -> Package_DIP:DIP-40_W15.24mm_Socket
- U18: value (none) -> YM2151; footprint (none) -> Package_DIP:DIP-24_W15.24mm_Socket
- U19: value (none) -> YM3012; footprint (none) -> Package_DIP:DIP-16_W7.62mm_Socket
- U2: value (none) -> SN7406; footprint (none) -> Package_DIP:DIP-14_W7.62mm_Socket
- U21: value (none) -> TL072; footprint (none) -> Package_DIP:DIP-8_W7.62mm_Socket
- U22: value (none) -> MCP7940N-xP; footprint (none) -> Package_DIP:DIP-8_W7.62mm
- U23: value (none) -> MercuryII-FPGA; footprint (none) -> JBCustoms:MercuryII_FPGA
- U3: value (none) -> SST39SF040; footprint (none) -> Socket:DIP_Socket-32_W11.9_W12.7_W15.24_W17.78_W18.5_3M_232-1285-00-0602J
- U4: value (none) -> AS6C1008-55PCN; footprint (none) -> Package_DIP:DIP-32_W15.24mm_Socket
- U5, U6, U7, U8: value (none) -> AS6C4008-55PCN; footprint (none) -> Package_DIP:DIP-32_W15.24mm_Socket
- U9: value (none) -> ATF1508; footprint (none) -> Package_LCC:PLCC-84_THT-Socket
- X1: value (none) -> 16mhz; footprint (none) -> Oscillator:Oscillator_DIP-8
- X3: value (none) -> 3.579545MHz; footprint (none) -> Oscillator:Oscillator_DIP-8
- Y1: value (none) -> 32.768KHz; footprint (none) -> Crystal:Crystal_C26-LF_D2.1mm_L6.5mm_Horizontal
Connections:
- net VPB: now also U9.74 (IO)
- no-connect marks 39 -> 38
