File: PCB/VeraHDMICard/vera-module-rev4.kicad_pcb (KiCad board)
At the start: 2 copper layers, 100 x 57.3 mm, 83 parts, among them J1 Conn_02x30_Odd_Even, J2 Prog, J3 HDMI_A_1.4, J4 Conn_01x02_Male, J5 AudioJack3, J6 Micro_SD_Card, J7 JTAG, U1 ICE40UP5K-SG48ITR50, U10 MIC5504-3.3YM5, U11 TFP410PAP, U12 SN74CB3T16210, U2 74AHC00PW, U4 74CBTLV3126PW,118, U6 WM8524CGEDT, U7 W25Q16JVSNIQ, U8 ATF1502AS-xAx44, U9 AP3417CKTR-G1, X1 SG5032CAN_25.000000M-TJGA3

Commit message: Updates
Other:
- net class Default removed
